File: KiCad/60ish_paska/60ish_paska.kicad_sch (KiCad schematic)
At the start: 155 parts, among them U1 ProMicro

Commit message: submoduling all folders KEKW
Parts:
- removed U1: ProMicro, symbol keebio:ProMicro
Changed lines of the file:
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@@
-    )
-  )
-  (symbol (lib_id "keebio:ProMicro") (at 43.18 46.99 0) (unit 1)
-    (in_bom yes) (on_board yes) (dnp no) (fields_autoplaced)
-    (property "Reference" "U1" (at 43.18 25.4 0)
-      (effects (font (size 1.524 1.524)))
-    )
-    (property "Value" "ProMicro" (at 43.18 27.94 0)
-      (effects (font (size 1.524 1.524)))
-    )
-    (property "Footprint" "" (at 69.85 110.49 90)
-      (effects (font (size 1.524 1.524)) hide)
-    )
-    (property "Datasheet" "" (at 69.85 110.49 90)
-      (effects (font (size 1.524 1.524)) hide)
-    )
-    (pin "1")
-    (pin "10")
-    (pin "11")
-    (pin "12")
-    (pin "13")
-    (pin "14")
-    (pin "15")
-    (pin "16")
-    (pin "17")
-    (pin "18")
-    (pin "19")
-    (pin "2")
-    (pin "20")
-    (pin "21")
-    (pin "22")
-    (pin "23")
-    (pin "24")
-    (pin "3")
-    (pin "4")
-    (pin "5")
-    (pin "6")
-    (pin "7")
-    (pin "8")
-    (pin "9")
-    (instances
-      (project "60ish_paska"
-        (path "/cd7d090e-7de8-4269-9296-a725237f24d2"
-          (reference "U1") (unit 1)
-        )
-      )
     )
   )
